File: hardware/radio/ethernet_poe.kicad_sch (KiCad schematic)
At the start: 59 parts, among them J301 DS1128-S80BP, T301 B1608S, U301 W5500, U401 DP9900LP-5V, Y301 X322525MOB4SI

Commit message: fix(hardware): apply the schematic review findings
Parts:
- added R402: 56R, freedo-radio:R_2512_6332Metric, symbol freedo-radio:R
- C318, C319, C320, C321: value 10nF -> 10nF/100V
- C322, C323: value 1nF -> 1nF/2kV
Connections:
- net +VDC: now also R402.1
- net GND: now also R402.2
Other:
- note added: "R402 DNP: fit if the PSE drops power at low load (DP9900 needs >= 100 mA)"

Commit message: feat(hardware): set up the board stackup, rules and outline
Connections:
- net TD_P: now reaches R304.2, R309.1, T301.1 (TD+)
- net TD_N: now reaches R305.2, R310.1, T301.3 (TD-)
- net RX_TERM_P: now reaches C315.2, R307.1, R311.1
- net RX_TERM_N: now reaches C316.2, R308.2, R312.1
- net RD_N: now reaches C316.1, T301.8 (RD-)
- net RD_P: now reaches C315.1, T301.6 (RD+)
- net MDI_1 renamed MDI_TX_P
- net MDI_2 renamed MDI_TX_N
- net MDI_3 renamed MDI_RX_P
- net MDI_6 renamed MDI_RX_N
Changed lines of the file:
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@@
 		)
 	)
-	(label "MDI_1"
+	(label "TD_P"
+		(at 152.4 55.88 0)
+		(effects
+			(font
+				(size 1.27 1.27)
+			)
+			(justify left bottom)
+		)
+	)
+	(label "TD_N"
+		(at 152.4 60.96 0)
+		(effects
+			(font
+				(size 1.27 1.27)
+			)
+			(justify left bottom)
+		)
+	)
+	(label "RD_P"
+		(at 152.4 66.04 0)
+		(effects
+			(font
+				(size 1.27 1.27)
+			)
+			(justify left bottom)
+		)
+	)
+	(label "RD_N"
+		(at 152.4 71.12 0)
+		(effects
+			(font
+				(size 1.27 1.27)
+			)
+			(justify left bottom)
+		)
+	)
+	(label "RX_TERM_P"
+		(at 186.69 81.28 90)
+		(effects
+			(font
+				(size 1.27 1.27)
+			)
+			(justify left bottom)
+		)
+	)
+	(label "RX_TERM_N"
+		(at 186.69 101.6 90)
+		(effects
+			(font
+				(size 1.27 1.27)
+			)
+			(justify left bottom)
+		)
+	)
+	(label "MDI_TX_P"
 		(at 40.64 54.61 0)
 		(effects
@@
 		)
 	)
-	(label "MDI_1"
+	(label "MDI_TX_P"
 		(at 127 55.88 180)
 		(effects
@@
 		)
 	)
-	(label "MDI_2"
+	(label "MDI_TX_N"
 		(at 40.64 57.15 0)
 		(effects
@@
 		)
 	)
-	(label "MDI_2"
+	(label "MDI_TX_N"
 		(at 127 60.96 180)
 		(effects
@@
 		)
 	)
-	(label "MDI_3"
+	(label "MDI_RX_P"
 		(at 40.64 59.69 0)
 		(effects
@@
 		)
 	)
-	(label "MDI_3"
+	(label "MDI_RX_P"
 		(at 127 66.04 180)
 		(effects
@@
 		)
 	)
-	(label "MDI_6"
+	(label "MDI_RX_N"
 		(at 40.64 67.31 0)
 		(effects
@@
 		)
 	)
-	(label "MDI_6"
+	(label "MDI_RX_N"
 		(at 127 71.12 180)
 		(effects

Commit message: feat(hardware): move the radio to the ebyte e07 module and fix the power review findings
Parts:
- C401: LCSC C72477 -> C264047; MPN RVT1E101M0607 -> EEHZA1E101XP
- J301: value DS1128-S80BP -> TM24RSG-5A-88; footprint freedo-radio:RJ45_CONNFLY_DS1128-S80BP -> freedo-radio:RJ45_Hirose_TM24RSG-5A-88; symbol freedo-radio:DS1128-S80BP -> freedo-radio:TM24RSG-5A-88; LCSC C86586 -> C6285250; MPN DS1128-S80BP -> TM24RSG-5A-88
Connections:
- net SHIELD: now also J301.11 (SHIELD), J301.12 (SHIELD), J301.13 (SHIELD), J301.14 (SHIELD)
Changed lines of the file:
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@@
   )
 	(symbol
-		(lib_id "freedo-radio:DS1128-S80BP")
+		(lib_id "freedo-radio:TM24RSG-5A-88")
 		(at 30.48 63.5 0)
 		(mirror y)
@@
 			)
 		)
-		(property "Value" "DS1128-S80BP"
+		(property "Value" "TM24RSG-5A-88"
 			(at 30.48 49.53 0)
 			(effects
@@
 			)
 		)
-		(property "Footprint" "freedo-radio:RJ45_CONNFLY_DS1128-S80BP"
+		(property "Footprint" "freedo-radio:RJ45_Hirose_TM24RSG-5A-88"
 			(at 30.48 63.5 0)
 			(hide yes)
@@
 			)
 		)
-		(property "Datasheet" "https://www.lcsc.com/datasheet/lcsc_datasheet_1811141110_CONNFLY-Elec-DS1128-S80BP_C86586.pdf"
+		(property "Datasheet" "https://www.lcsc.com/datasheet/lcsc_datasheet_2407051755_HRS-Hirose-TM24RSG-5A-88_C6285250.pdf"
 			(at 30.48 63.5 0)
 			(hide yes)
@@
 			)
 		)
-		(property "Description" "CONNFLY RJ45 8P8C, shielded, no LEDs, THT. Pins 9/10 = shield."
+		(property "Description" "Hirose TM24RSG-5A-88 RJ45 8P8C, shielded, tab up, no LEDs, THT, 1500 V AC terminal to shield (TM24R catalog p.2). Pins 9-14 = shield: 9/10 front shell, 12/14 rear shell, 11/13 ground springs (11-14 hidden, stacked under 9/10)."
 			(at 30.48 63.5 0)
 			(hide yes)
@@
 			)
 		)
-		(property "MPN" "DS1128-S80BP"
+		(property "MPN" "TM24RSG-5A-88"
 			(at 30.48 63.5 0)
 			(hide yes)
@@
 			)
 		)
-		(property "LCSC" "C86586"
+		(property "LCSC" "C6285250"
 			(at 30.48 63.5 0)
 			(hide yes)
@@
 			)
 		)
-		(property "MPN" "RVT1E101M0607"
+		(property "MPN" "EEHZA1E101XP"
 			(at 172.72 217.17 0)
 			(hide yes)
@@
 			)
 		)
-		(property "LCSC" "C72477"
+		(property "LCSC" "C264047"
 			(at 172.72 217.17 0)
 			(hide yes)
