File: hardware/radio/usb_power.kicad_sch (KiCad schematic)
At the start: 15 parts, among them J201 TYPE-C-31-M-12, U202 USBLC6-2SC6, U203 LDL1117S33R

Commit message: fix(hardware): apply the schematic review findings
Parts:
- added C208: 100nF, freedo-radio:C_0603_1608Metric, symbol freedo-radio:C
- added R215: 10k, freedo-radio:R_0603_1608Metric, symbol freedo-radio:R
Connections:
- net GND: now also C208.2, R215.2
- net VBUS: now also C208.1, R215.1

Commit message: feat(hardware): move the radio to the ebyte e07 module and fix the power review findings
Parts:
- removed U202: USBLC6-2SC6, freedo-radio:SOT-23-6_L2.9-W1.6-P0.95-LS2.8-BL, symbol freedo-radio:USBLC6-2SC6
- added C209: 100nF, freedo-radio:C_0603_1608Metric, symbol freedo-radio:C
- added R216: 68k, freedo-radio:R_0603_1608Metric, symbol freedo-radio:R
- added R217: 100k, freedo-radio:R_0603_1608Metric, symbol freedo-radio:R
- added U202: H5VUT2U, freedo-radio:SOT-23-3_L2.9-W1.5-P1.90-LS2.6-BR, symbol freedo-radio:H5VUT2U
- C202: value 22uF -> 10uF; LCSC C45783 -> C15850; MPN CL21A226MAQNNNE -> CL21A106KAYNNNE
- D201: value SMF5.0A -> SMF6.0A; symbol freedo-radio:SMF5.0A -> freedo-radio:SMF6.0A; LCSC C19077497 -> C19077499; MPN SMF5.0A -> SMF6.0A
- R215: value 10k -> 4.7k; LCSC C25804 -> C23162; MPN 0603WAF1002T5E -> 0603WAF4701T5E
- U203: value LDL1117S33R -> TLV76133DCYR; symbol freedo-radio:LDL1117S33R -> freedo-radio:TLV76133DCYR; LCSC C435835 -> C7527500; MPN LDL1117S33R -> TLV76133DCYR
Connections:
- net GND: now also C209.2, R217.2, U202.3 (GND)
- net USB_DN: now also U202.1 (I/O1)
- net USB_DP: now also U202.2 (I/O2)
- net VBUS: now also R216.1
- new net VBUS_SENSE: C209.1, R216.2, R217.1
Other:
- note added: "C209: tau 4 ms, the pin stays below VDD + 0.3 V during the 7.1 V hot-plug peak."
- note added: "U202 at J201 (no VBUS pin: no path from the D+ pull-up to VBUS, review E03)"
- note added: "U203: tab on >= 4 cm2 top copper, >= 8 vias to a 3V3 pour on B.Cu (spec 4.4) C202, C203 at IN; C204, C205 at OUT (TLV761 DS 7.3)"
- note added: "VBUS_SENSE = 0.595 x VBUS: 2.62 V at 4.40 V, 3.27 V at 5.5 V (spec 5.2)."
- note removed: "U202 at the connector"
- note removed: "U203: tab on >= 2 cm2 copper + >= 6 vias (spec 4.4) C202, C203 at VIN; C204, C205 at VOUT (LDL1117 DS 6.2)"
