File: hardware/radio/freedo-radio.kicad_pcb (KiCad board)
At the start: 4 copper layers, 100 x 75 mm, 132 parts, among them J1 SMA-KE-347-H13.5-1.6, J201 TYPE-C-31-M-12, J203 GPIO, J301 TM24RSG-5A-88, SW201 TS-1187A-B-A-B, SW202 TS-1187A-B-A-B, T301 B1608S, U1 E07-900MM10S, U201 ESP32-S3-MINI-1-N8, U202 H5VUT2U, U203 TLV76133DCYR, U301 W5500, U401 DP9900LP-5V, Y301 X322525MOB4SI

Commit message: fix(hardware): apply the routed-board review fixes
Parts:
- added FID1: Fiducial, freedo-radio:Fiducial_1mm_Mask2mm, F.Cu at (200.5, 53.5)
- added FID2: Fiducial, freedo-radio:Fiducial_1mm_Mask2mm, F.Cu at (284.0, 70.5)
- added FID3: Fiducial, freedo-radio:Fiducial_1mm_Mask2mm, F.Cu at (280.5, 121.5)
- TP101, TP102, TP103, TP104, TP105, TP106, TP107: footprint freedo-radio:TestPoint_Pad_D1.5mm -> freedo-radio:TestPoint_THTPad_D1.5mm_Drill0.7mm
- moved TP101 25.1 mm to (263.3, 80.4)
- moved TP104 25.1 mm to (263.3, 82.9)
- moved TP106 25.1 mm to (263.3, 75.3)
- moved TP105 25.1 mm to (263.3, 77.8)
- moved TP107 10.7 mm to (279.0, 76.9)
- moved TP102 8.46 mm to (279.0, 79.5)
- moved TP103 8.46 mm to (279.0, 82.0)
- moved SW201 1.90 mm to (270.6, 55.1), turned to 180 degrees
- moved SW202 1.90 mm to (278.7, 55.1), turned to 180 degrees
- moved R206 1.25 mm to (278.7, 58.5)
- moved R207 0.50 mm to (265.3, 57.0)
- moved R301 0.36 mm to (247.2, 80.7), turned to 90 degrees
- moved R203 0.07 mm to (254.2, 69.6)
- moved R204 0.07 mm to (256.2, 69.6)
- moved C316 0.05 mm to (221.2, 71.3)
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Routing:
- net /mcu/CC_GDO2: track 78.7 -> 52.3 mm, vias 2 -> 0
- net /mcu/CC_GDO0: track 72.8 -> 48.2 mm, vias 2 -> 1
- net /mcu/CC_CSN: track 66.3 -> 47.2 mm, vias 3 -> 2
- net /mcu/CC_SCK: track 55.2 -> 39.9 mm, vias 2 -> 1
- net /ethernet_poe/3V3A: track 53.7 -> 68.1 mm, vias 0 -> 5
- net /mcu/CC_MOSI: track 55.6 -> 44.4 mm, vias 2 -> 1
- net /mcu/CC_MISO: track 53.5 -> 43.3 mm, vias 2 -> 1
- net /mcu/E22_NRST: track 55.8 -> 51.7 mm
- net /mcu/BOOT: track 37.3 -> 40.7 mm
- net /ethernet_poe/TXN: track 21.7 -> 19.0 mm
- net /ethernet_poe/TD_N: track 8.40 -> 10.7 mm
- net /ethernet_poe/MDI_RX_N: track 17.9 -> 20.1 mm
- net /ethernet_poe/MDI_RX_P: track 18.1 -> 20.1 mm
- net GND: track 62.3 -> 60.9 mm, vias 551 -> 562
- net /mcu/EN: track 13.6 -> 12.9 mm
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- removed copper zone on F.Cu, net /ethernet_poe/3V3A
Other:
- board text added: "3V3A B.Cu trunk to the AVDD capacitors"
- board text added: "TX/RX to J203: B.Cu under U201, then along the top edge"
- board text added: "radio test pads: GDO2 F.Cu, the rest one via + B.Cu"
- board text removed: "3V3 pour to U301"
- board text removed: "TX/RX to J203, B.Cu under U201"
- board text removed: "radio TP stubs, B.Cu"
